File: adega_iot.kicad_sch (KiCad schematic)
At the start: 66 parts, among them J1 Conn_01x03_Pin, J2 Conn_01x02_Pin, J3 Screw_Terminal_01x02, J4 Conn_01x03_Pin, J6 Conn_01x03_Pin, J7 Screw_Terminal_01x02, J8 Conn_01x02_Pin, J9 Conn_01x02_Pin, Q1 BC548, Q10 BC548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

Commit message: bug fixes
Connections:
- net BOOT: no longer names the net of U2.25 (GPIO0/BOOT/ADC2_CH1)
- no-connect marks 14 -> 15
Changed lines of the file:
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@@
   (no_connect (at 48.26 59.69))
   (no_connect (at 114.3 87.63))
+  (no_connect (at 114.3 52.07))
   (no_connect (at 114.3 62.23))
   (no_connect (at 114.3 97.79))
@@
     (stroke (width 0) (type default))
   )
-  (wire (pts (xy 114.3 52.07) (xy 130.81 52.07))
-    (stroke (width 0) (type default))
-  )
   (wire (pts (xy 21.59 121.92) (xy 19.05 121.92))
     (stroke (width 0) (type default))
@@
     (effects (font (size 1.27 1.27)) (justify left bottom))
   )
-  (label "BOOT" (at 124.46 52.07 0) (fields_autoplaced)
-    (effects (font (size 1.27 1.27)) (justify left bottom))
-  )
